File: batt.sch (KiCad schematic (older format))
At the start: 14 parts

Commit message: workin on the sheetz
Parts:
- removed Q?: MOSFET_P, ~, symbol MOSFET_P
- added BT?: BATTERY, ~, symbol BATTERY
- added C? (x2): 10uF (0.3 ESR MAX), ~, symbol CSMALL
- added C?: 0.1uF, ~, symbol CSMALL
- added D?: DIODESCH, ~, symbol DIODESCH
- added Q? (x2): AON2400, ~, symbol AON2400
- added R?: R, ~, symbol R
- added R? (x2): 1K, ~, symbol R
- added U?: AAA-, ~, symbol TOUCHPAD
- added U?: AAA+, ~, symbol TOUCHPAD
- added U?: LM2767, symbol LM2767
- added U?: MMA8653FC, symbol MMA8653FC
- added U?: C8051T606, symbol C8051T606
Connections:
- net labels removed: GND, VDD
- wire segments 34 -> 72
- no-connect marks 0 -> 8
Other:
- note added: "3V (or if doubler fails, V_BATT - V_DIODE)\n"
- note added: "Actual Implementation"
- note added: "Debug Implementation"
- note added: "LOCAL GND"
- note added: "Push-pull"
- note added: "input"
- note added: "output"
- note added: "weak pull-up"
- note removed: "0V"
- note removed: "3V\n"
- moved on the sheet: BT?, R?

Commit message: finalizing schematic
nicely organized hierarchachylhclhylllyy
Parts:
- removed BT? (x2): BATTERY, ~, symbol BATTERY
- removed C? (x4): 10uF (0.3 ESR MAX), ~, symbol CSMALL
- removed C? (x2): 0.1uF, ~, symbol CSMALL
- removed D? (x2): DIODESCH, ~, symbol DIODESCH
- removed Q? (x2): AON2400, ~, symbol AON2400
- removed R? (x2): R, ~, symbol R
- removed R? (x4): 1K, ~, symbol R
- removed U? (x2): AAA-, ~, symbol TOUCHPAD
- removed U? (x2): AAA+, ~, symbol TOUCHPAD
- removed U? (x2): LM2767, symbol LM2767
- removed U? (x2): MMA8653FC, symbol MMA8653FC
- removed U? (x2): C8051T606, symbol C8051T606
Connections:
- net labels removed: 2xV_BATT, INT1, INT2, SCL, SDA, V_BATT
- wire segments 72 -> 14
- no-connect marks 8 -> 0
Other:
- note added: "Debug Circuit"
- note added: "Desired circuit"
- note removed: "0.9V <-> 1.5V"
- note removed: "3V (or if doubler fails, V_BATT - V_DIODE)\n"
- note removed: "Actual Implementation"
- note removed: "Debug Implementation"
- note removed: "LOCAL GND"
- note removed: "Push-pull"
- note removed: "input"
- note removed: "output"
- note removed: "weak pull-up"
