File: proc_MSP430G2203.sch (KiCad schematic (older format))
At the start: 0 parts

Commit message: finalizing schematic
nicely organized hierarchachylhclhylllyy
Parts:
- added U?: MSP430G2203IPW28, ~, symbol MSP430G2203IPW28
Connections:
- new net FET_CTRL: U?.10 (P2.0/TA1.0)
- new net GND: U?.28 (DVSS)
- new net INT1: U?.11 (P2.1/TA1.1)
- new net INT2: U?.12 (P2.2/TA1.1)
- new net SCL: U?.22 (P1.6/TA0.1/A6/UCB0SOMI/UCB0SCL/TDI/TCLK)
- new net SDA: U?.23 (P1.7/A7/UCB0SIMO/UCB0SDA/TDO/TDI)
- new net VDD: U?.1 (DVCC)
Changed lines of the file:
@@
 $Descr A4 11693 8268
 encoding utf-8
-Sheet 1 3
+Sheet 3 5
 Title ""
-Date "14 oct 2014"
+Date "15 oct 2014"
 Rev ""
 Comp ""
@@
 Comment4 ""
 $EndDescr
+Text HLabel 4100 3100 0    60   Input ~ 0
+VDD
+Text HLabel 4100 4750 0    60   Input ~ 0
+GND
+Text HLabel 4100 4100 0    60   Output ~ 0
+SDA
+Text HLabel 4100 4000 0    60   Output ~ 0
+SCL
+Text HLabel 7900 3200 2    60   Input ~ 0
+INT1
+Text HLabel 7900 3300 2    60   Input ~ 0
+INT2
+Text HLabel 7900 3100 2    60   Output ~ 0
+FET_CTRL
+$Comp
+L MSP430G2203IPW28 U?
+U 1 1 543E080C
+P 6000 3000
+F 0 "U?" H 6000 3050 60  0000 C CNN
+F 1 "MSP430G2203IPW28" H 6000 1200 60  0000 C CNN
+F 2 "~" H 5950 3000 60  0000 C CNN
+F 3 "~" H 5950 3000 60  0000 C CNN
+	1    6000 3000
+	1    0    0    -1
+$EndComp
+Wire Wire Line
+	4100 3100 4200 3100
+Wire Wire Line
+	4100 4000 4200 4000
+Wire Wire Line
+	4100 4100 4200 4100
+Wire Wire Line
+	4100 4750 4200 4750
+Wire Wire Line
+	7800 3100 7900 3100
+Wire Wire Line
+	7800 3200 7900 3200
+Wire Wire Line
+	7800 3300 7900 3300
 $EndSCHEMATC
